Commit message: 202007171715

File: src/ur5_gripper/urdf/ur5_rg2_gripper.xacro (robot description, xacro)
@@ -27,5 +27,5 @@
     <parent link="world" />
     <child link = "base_link" />
-    <origin xyz="0.0 0.0 0.0" rpy="0.0 0.0 0.0" />
+    <origin xyz="0.0 0.0 0.998" rpy="0.0 0.0 0.0" />
   </joint>
 </robot>
