Commit message: gazebo object abandoned

File: src/ur5_gripper/urdf/ur5_simple_gripper.xacro (robot description, xacro)
@@ -29,5 +29,5 @@
     <parent link="world" />
     <child link = "base_link" />
-    <origin xyz="0.0 0.0 0.998" rpy="0.0 0.0 0.0" />
+    <origin xyz="0.0 0.0 1.0" rpy="0.0 0.0 0.0" />
   </joint>
 </robot>
