Commit message: af85 fixed

File: src/bo_ur5/urdf/robotiq_coupler.xacro (robot description, xacro)
@@ -5,5 +5,6 @@
       <parent link="${connected_to}" />
       <child link="${prefix}robotiq_coupler_link" />
-      <origin xyz="0 0 0.004" rpy="0 0 ${-pi/2.0}" />
+      <!--      <origin xyz="0 0 0" rpy="0 0 ${-pi/2.0}" /> -->
+      <origin xyz="0 0 0" rpy="0 0 0" />
     </joint>
     <link name="${prefix}robotiq_coupler_link">
@@ -27,9 +28,9 @@
 	<mu1> 0.9 </mu1>
 	<mu2> 0.9 </mu2>
-	<material>Gazebo/FlatBlack</material>
+	<material>Gazebo/FlatWhite</material>
       </gazebo>
     </link>
     <joint name="${prefix}gripper_joint" type="fixed">
-      <origin xyz="0 0 0.008" rpy="0 0 0" />
+      <origin xyz="0 0 0" rpy="0 0 0" />
       <parent link="${prefix}robotiq_coupler_link" />
       <child link="${prefix}robotiq_arg2f_base_link" />

File: src/robotiq_2f_85_gripper_visualization/urdf/robotiq_arg2f.xacro (robot description, xacro)
@@ -11,5 +11,5 @@
         <origin xyz="0 0 0" rpy="0 0 0" />
         <geometry>
-          <mesh filename="package://robotiq_2f_85_gripper_visualization/meshes/visual/robotiq_arg2f_85_base_link.dae" scale="0.001 0.001 0.001"/>
+          <mesh filename="package://robotiq_2f_85_gripper_visualization/meshes/collision/robotiq_arg2f_85_base_link.stl" scale="1 1 1"/>
         </geometry>
         <material name="">

File: src/robotiq_2f_85_gripper_visualization/urdf/robotiq_arg2f_85_model_macro.xacro (robot description, xacro)
@@ -136,5 +136,5 @@
       <child link="${prefix}${fingerprefix}_inner_knuckle" />
       <axis xyz="1 0 0" />
-      <limit lower="0" upper="0.8757" velocity="2.0" effort="1000" />
+      <limit lower="-0.8757" upper="0.8757" velocity="2.0" effort="1000" />
       <mimic joint="${prefix}finger_joint" multiplier="1" offset="0" />
     </joint>
@@ -175,5 +175,5 @@
       <child link="${prefix}right_outer_knuckle" />
       <axis xyz="1 0 0" />
-      <limit lower="0" upper="0.81" velocity="2.0" effort="1000" />
+      <limit lower="-0.81" upper="0.81" velocity="2.0" effort="1000" />
       <mimic joint="${prefix}finger_joint" multiplier="1" offset="0" />
     </joint>
