Commit message: bo ur53 moveit config deleted

File: src/robotiq/robotiq_2f_model/model/robotiq_2f_85_original.urdf.xacro (robot description, xacro)
@@ -1,4 +1,3 @@
 <?xml version="1.0"?>
-<!-- revolute joints have been replaced to 'fixed' joint for the stability in GAZEBO (chester -->
 <!--
 	Coordinate system convention for grippers:
@@ -61,5 +60,5 @@
 		</link>
 		<!-- right finger -->
-		<joint name="${name}_right_driver_joint" type="fixed">
+		<joint name="${name}_right_driver_joint" type="revolute">
 			<origin xyz="0 0.0306011 0.054904" rpy="0 0 0"/>
 			<parent link="${name}_base"/>
@@ -103,5 +102,5 @@
 		</xacro:unless>
 		<xacro:if value="${adaptive_transmission}">
-			<joint name="${name}_right_coupler_joint" type="fixed">
+			<joint name="${name}_right_coupler_joint" type="revolute">
 			<origin xyz="0 0.0315 -0.0041" rpy="0 0 0"/>
 			<parent link="${name}_right_driver"/>
@@ -138,5 +137,5 @@
 			</xacro:if>
 		</link>
-		<joint name="${name}_right_follower_joint" type="fixed">
+		<joint name="${name}_right_follower_joint" type="revolute">
 			<origin xyz="0 0.0061 0.0471" rpy="0 0 0"/>
 			<parent link="${name}_right_coupler"/>
@@ -208,5 +207,5 @@
 			</link>
 		</xacro:if>
-		<joint name="${name}_right_spring_link_joint" type="fixed">
+		<joint name="${name}_right_spring_link_joint" type="revolute">
 			<origin xyz="0 0.012 0.0614" rpy="0 0 0"/>
 			<parent link="${name}_base"/>
@@ -246,5 +245,5 @@
 		</link>
 		<!-- left finger -->
-		<joint name="${name}_left_driver_joint" type="fixed">
+		<joint name="${name}_left_driver_joint" type="revolute">
 			<origin xyz="0 -0.0306011 0.054904" rpy="0 0 3.141592653589793"/>
 			<parent link="${name}_base"/>
@@ -291,5 +290,5 @@
 		</xacro:unless>
 		<xacro:if value="${adaptive_transmission}">
-			<joint name="${name}_left_coupler_joint" type="fixed">
+			<joint name="${name}_left_coupler_joint" type="revolute">
 			<origin xyz="0 0.0315 -0.0041" rpy="0 0 0"/>
 			<parent link="${name}_left_driver"/>
@@ -326,5 +325,5 @@
 			</xacro:if>
 		</link>
-		<joint name="${name}_left_follower_joint" type="fixed">
+		<joint name="${name}_left_follower_joint" type="revolute">
 			<origin xyz="0 0.0061 0.0471" rpy="0 0 0"/>
 			<parent link="${name}_left_coupler"/>
@@ -396,5 +395,5 @@
 			</link>
 		</xacro:if>
-		<joint name="${name}_left_spring_link_joint" type="fixed">
+		<joint name="${name}_left_spring_link_joint" type="revolute">
 			<origin xyz="0 -0.012 0.0614" rpy="0 0 3.141592653589793"/>
 			<parent link="${name}_base"/>
