Commit message: code refactored to cope with robotiq af85 stable edition

File: src/bo_ur5e/urdf/ur5e_af85.urdf.xacro (robot description, xacro)
@@ -8,7 +8,7 @@
   <xacro:include filename="$(find ur_e_description)/urdf/ur5e.urdf.xacro" />
   <!-- robotiq coupler -->
-  <xacro:include filename="robotiq_coupler.xacro" />
+  <xacro:include filename="$(find robotiq_2f_model)/model/robotiq_ur_coupler.urdf.xacro" />
   <!-- robotiq_85_model -->
-  <xacro:include filename="$(find robotiq_2f_85_gripper_visualization)/urdf/robotiq_arg2f_85_model_macro.xacro" />
+  <xacro:include filename="$(find robotiq_2f_model)/model/robotiq_2f_85.urdf.xacro" />
   <!-- arm -->
   <xacro:ur5e_robot prefix="" joint_limited="true"
@@ -20,6 +20,8 @@
     wrist_3_lower_limit="${-pi}" wrist_3_upper_limit="${pi}"
     />
-  <xacro:robotiq_coupler prefix="" connected_to="tool0" />
-  <xacro:robotiq_arg2f_85 prefix="" />
+  <xacro:robotiq_ur_coupler parent="tool0" name="tool1" />
+  <xacro:robotiq_2f_85 name="simple_gripper" parent="tool1" precise_collision="false" adaptive_transmission="false">
+    <origin xyz="0 0 0" rpy="0 0 0" />
+  </xacro:robotiq_2f_85>
   <link name="world" />
   <joint name="world_joint" type="fixed">
@@ -28,3 +30,8 @@
     <origin xyz="0.0 0.0 0.0" rpy="0.0 0.0 0.0" />
   </joint>
+  <gazebo>
+    <plugin name="gazebo_ros_control" filename="libgazebo_ros_control.so">
+      <robotNamespace>/</robotNamespace>
+    </plugin>
+  </gazebo>
 </robot>

Commit message: 20200724_1500

File: src/bo_ur5e/urdf/ur5e_af85.urdf.xacro (robot description, xacro)
@@ -32,5 +32,6 @@
   <gazebo>
     <plugin name="gazebo_ros_control" filename="libgazebo_ros_control.so">
-      <robotNamespace>/</robotNamespace>
+    </plugin>
+    <plugin name="gazebo_mimic_joint" filename="libroboticsgroup_gazebo_mimic_joint_plugin.so">
     </plugin>
   </gazebo>

File: src/robotiq/robotiq_2f_model/model/robotiq_2f_85.urdf.xacro (robot description, xacro)
@@ -1,4 +1,3 @@
 <?xml version="1.0"?>
-<!-- revolute joints have been replaced to 'fixed' joint for the stability in GAZEBO (chester -->
 <!--
 	Coordinate system convention for grippers:
@@ -33,7 +32,7 @@
 			</inertial>
 			<visual>
-				<origin xyz="0 0 0" rpy="0 -1.5708 0"/>
-				<geometry>
-					<mesh filename="package://robotiq_2f_model/model/meshes/2f85/visual/base.dae"/>
+				<origin xyz="0 0 0" rpy="0 0 0"/>
+				<geometry>
+					<mesh filename="package://robotiq_2f_model/model/meshes/2f85/collision/base.stl" scale="0.001 0.001 0.001"/>
 				</geometry>
 			</visual>
@@ -61,5 +60,5 @@
 		</link>
 		<!-- right finger -->
-		<joint name="${name}_right_driver_joint" type="fixed">
+		<joint name="${name}_right_driver_joint" type="revolute">
 			<origin xyz="0 0.0306011 0.054904" rpy="0 0 0"/>
 			<parent link="${name}_base"/>
@@ -103,5 +102,5 @@
 		</xacro:unless>
 		<xacro:if value="${adaptive_transmission}">
-			<joint name="${name}_right_coupler_joint" type="fixed">
+			<joint name="${name}_right_coupler_joint" type="revolute">
 			<origin xyz="0 0.0315 -0.0041" rpy="0 0 0"/>
 			<parent link="${name}_right_driver"/>
@@ -138,5 +137,5 @@
 			</xacro:if>
 		</link>
-		<joint name="${name}_right_follower_joint" type="fixed">
+		<joint name="${name}_right_follower_joint" type="revolute">
 			<origin xyz="0 0.0061 0.0471" rpy="0 0 0"/>
 			<parent link="${name}_right_coupler"/>
@@ -208,5 +207,5 @@
 			</link>
 		</xacro:if>
-		<joint name="${name}_right_spring_link_joint" type="fixed">
+		<joint name="${name}_right_spring_link_joint" type="revolute">
 			<origin xyz="0 0.012 0.0614" rpy="0 0 0"/>
 			<parent link="${name}_base"/>
@@ -246,5 +245,5 @@
 		</link>
 		<!-- left finger -->
-		<joint name="${name}_left_driver_joint" type="fixed">
+		<joint name="${name}_left_driver_joint" type="revolute">
 			<origin xyz="0 -0.0306011 0.054904" rpy="0 0 3.141592653589793"/>
 			<parent link="${name}_base"/>
@@ -291,5 +290,5 @@
 		</xacro:unless>
 		<xacro:if value="${adaptive_transmission}">
-			<joint name="${name}_left_coupler_joint" type="fixed">
+			<joint name="${name}_left_coupler_joint" type="revolute">
 			<origin xyz="0 0.0315 -0.0041" rpy="0 0 0"/>
 			<parent link="${name}_left_driver"/>
@@ -326,5 +325,5 @@
 			</xacro:if>
 		</link>
-		<joint name="${name}_left_follower_joint" type="fixed">
+		<joint name="${name}_left_follower_joint" type="revolute">
 			<origin xyz="0 0.0061 0.0471" rpy="0 0 0"/>
 			<parent link="${name}_left_coupler"/>
@@ -396,5 +395,5 @@
 			</link>
 		</xacro:if>
-		<joint name="${name}_left_spring_link_joint" type="fixed">
+		<joint name="${name}_left_spring_link_joint" type="revolute">
 			<origin xyz="0 -0.012 0.0614" rpy="0 0 3.141592653589793"/>
 			<parent link="${name}_base"/>

Commit message: 20200724_1510

File: src/bo_ur5e/urdf/ur5e_af85.urdf.xacro (robot description, xacro)
@@ -22,5 +22,5 @@
   <xacro:robotiq_ur_coupler parent="tool0" name="tool1" />
   <xacro:robotiq_2f_85 name="simple_gripper" parent="tool1" precise_collision="false" adaptive_transmission="false">
-    <origin xyz="0 0 0" rpy="0 0 0" />
+    <origin xyz="0 0 0" rpy="0 0 -${pi/2}" />
   </xacro:robotiq_2f_85>
   <link name="world" />
