Commit message: robotiq85 fixed points added

File: src/robotiq_85_gripper-master/robotiq_85_description/urdf/robotiq_85_gripper.urdf.xacro (robot description, xacro)
@@ -1,3 +1,4 @@
 <?xml version="1.0"?>
+<!-- Chester changed some of the parts of joint attribute to 'fixed' from 'continuous' for a longer time stability in GAZEBO... -->
 <robot name="robotiq_85_gripper" xmlns:xacro="http://ros.org/wiki/xacro">
     <xacro:include filename="$(find robotiq_85_description)/urdf/robotiq_85_gripper.transmission.xacro" />
@@ -35,5 +36,6 @@
             <limit lower="0.0" upper="0.804" velocity="2.0" effort="1000"/>
         </joint>
-        <joint name="${prefix}robotiq_85_right_knuckle_joint" type="continuous">
+	<!-- chester changed it to fixed -->
+        <joint name="${prefix}robotiq_85_right_knuckle_joint" type="fixed">
             <parent link="${prefix}robotiq_85_base_link"/>
             <child link="${prefix}robotiq_85_right_knuckle_link"/>
@@ -81,10 +83,12 @@
             </inertial>
         </link>
-        <joint name="${prefix}robotiq_85_left_finger_joint" type="continuous">
+	<!-- chester changed it to fixed -->
+        <joint name="${prefix}robotiq_85_left_finger_joint" type="fixed">
             <parent link="${prefix}robotiq_85_left_knuckle_link"/>
             <child link="${prefix}robotiq_85_left_finger_link"/>
             <origin xyz="-0.00408552455 -0.03148604435 0.0" rpy="0 0 0" />
         </joint>
-        <joint name="${prefix}robotiq_85_right_finger_joint" type="continuous">
+	<!-- chester changed it to fixed -->
+        <joint name="${prefix}robotiq_85_right_finger_joint" type="fixed">
             <parent link="${prefix}robotiq_85_right_knuckle_link"/>
             <child link="${prefix}robotiq_85_right_finger_link"/>
@@ -129,5 +133,6 @@
             </inertial>
         </link>
-        <joint name="${prefix}robotiq_85_left_inner_knuckle_joint" type="continuous">
+	<!-- chester changed it to fixed -->
+        <joint name="${prefix}robotiq_85_left_inner_knuckle_joint" type="fixed">
             <parent link="${prefix}robotiq_85_base_link"/>
             <child link="${prefix}robotiq_85_left_inner_knuckle_link"/>
@@ -137,5 +142,6 @@
             <mimic joint="${prefix}robotiq_85_left_knuckle_joint" offset="0"/>
         </joint>
-        <joint name="${prefix}robotiq_85_right_inner_knuckle_joint" type="continuous">
+	<!-- chester changed it to fixed -->
+        <joint name="${prefix}robotiq_85_right_inner_knuckle_joint" type="fixed">
             <parent link="${prefix}robotiq_85_base_link"/>
             <child link="${prefix}robotiq_85_right_inner_knuckle_link"/>
@@ -183,5 +189,6 @@
             </inertial>
         </link>
-        <joint name="${prefix}robotiq_85_left_finger_tip_joint" type="continuous">
+	<!-- chester changed it to fixed -->
+        <joint name="${prefix}robotiq_85_left_finger_tip_joint" type="fixed">
             <parent link="${prefix}robotiq_85_left_inner_knuckle_link"/>
             <child link="${prefix}robotiq_85_left_finger_tip_link"/>
@@ -191,5 +198,6 @@
             <mimic joint="${prefix}robotiq_85_left_knuckle_joint" multiplier="-1"/>
         </joint>
-        <joint name="${prefix}robotiq_85_right_finger_tip_joint" type="continuous">
+	<!-- chester changed it to fixed -->
+        <joint name="${prefix}robotiq_85_right_finger_tip_joint" type="fixed">
             <parent link="${prefix}robotiq_85_right_inner_knuckle_link"/>
             <child link="${prefix}robotiq_85_right_finger_tip_link"/>

File: src/ur5_gripper/urdf/ur5_simple_gripper.xacro (robot description, xacro)
@@ -8,7 +8,7 @@
   <xacro:include filename="$(find ur_description)/urdf/ur5.urdf.xacro" />
   <!-- robotiq coupler -->
-  <xacro:include filename="robotiq_coupler.xacro" />
+  <xacro:include filename="$(find robotiq_2f_model)/model/robotiq_ur_coupler.urdf.xacro" />
   <!-- robotiq_85_model -->
-  <xacro:include filename="$(find robotiq_2f_model)/model/robotiq_2f_85.urdf.xacro" />
+  <xacro:include filename="$(find robotiq_85_description)/urdf/robotiq_85_gripper.urdf.xacro" />
   <!-- arm -->
   <xacro:ur5_robot prefix="" joint_limited="true"
@@ -21,13 +21,13 @@
     transmission_hw_interface="$(arg transmission_hw_interface)"
     />
-  <xacro:robotiq_coupler prefix="" connected_to="tool0" />
-  <xacro:robotiq_2f_85 name="simple_gripper" parent="tool1" precise_collision="false" adaptive_transmission="false">
-                <origin xyz="0 0 0" rpy="0 0 0"/>
-  </xacro:robotiq_2f_85>
+  <xacro:robotiq_ur_coupler parent="tool0" name="tool1" />
+  <xacro:robotiq_85_gripper prefix="" parent="tool1" >
+                <origin xyz="0 0 0" rpy="${pi/2} -${pi/2} 0"/>
+  </xacro:robotiq_85_gripper>
   <link name="world" />
   <joint name="world_joint" type="fixed">
     <parent link="world" />
     <child link = "base_link" />
-    <origin xyz="0.0 0.0 0.0" rpy="0.0 0.0 0.0" />
+    <origin xyz="0.0 0.0 0.998" rpy="0.0 0.0 0.0" />
   </joint>
 </robot>
