Commit message: robotiq_85_gripper_static consideration has been applied

File: src/robotiq_85_gripper-master/robotiq_85_description/urdf/robotiq_85_gripper_static.urdf.xacro (robot description, xacro)
@@ -1,3 +1,4 @@
 <?xml version="1.0"?>
+<!-- Chester changed some of the parts of joint attribute to 'fixed' from 'continuous' for a longer time stability in GAZEBO... -->
 <robot name="robotiq_85_gripper" xmlns:xacro="http://ros.org/wiki/xacro">
     <xacro:include filename="$(find robotiq_85_description)/urdf/robotiq_85_gripper.transmission.xacro" />
@@ -35,5 +36,6 @@
             <limit lower="0.0" upper="0.804" velocity="2.0" effort="1000"/>
         </joint>
-        <joint name="${prefix}robotiq_85_right_knuckle_joint" type="continuous">
+	<!-- chester changed it to fixed -->
+        <joint name="${prefix}robotiq_85_right_knuckle_joint" type="fixed">
             <parent link="${prefix}robotiq_85_base_link"/>
             <child link="${prefix}robotiq_85_right_knuckle_link"/>
@@ -81,10 +83,12 @@
             </inertial>
         </link>
-        <joint name="${prefix}robotiq_85_left_finger_joint" type="continuous">
+	<!-- chester changed it to fixed -->
+        <joint name="${prefix}robotiq_85_left_finger_joint" type="fixed">
             <parent link="${prefix}robotiq_85_left_knuckle_link"/>
             <child link="${prefix}robotiq_85_left_finger_link"/>
             <origin xyz="-0.00408552455 -0.03148604435 0.0" rpy="0 0 0" />
         </joint>
-        <joint name="${prefix}robotiq_85_right_finger_joint" type="continuous">
+	<!-- chester changed it to fixed -->
+        <joint name="${prefix}robotiq_85_right_finger_joint" type="fixed">
             <parent link="${prefix}robotiq_85_right_knuckle_link"/>
             <child link="${prefix}robotiq_85_right_finger_link"/>
@@ -129,5 +133,6 @@
             </inertial>
         </link>
-        <joint name="${prefix}robotiq_85_left_inner_knuckle_joint" type="continuous">
+	<!-- chester changed it to fixed -->
+        <joint name="${prefix}robotiq_85_left_inner_knuckle_joint" type="fixed">
             <parent link="${prefix}robotiq_85_base_link"/>
             <child link="${prefix}robotiq_85_left_inner_knuckle_link"/>
@@ -137,5 +142,6 @@
             <mimic joint="${prefix}robotiq_85_left_knuckle_joint" offset="0"/>
         </joint>
-        <joint name="${prefix}robotiq_85_right_inner_knuckle_joint" type="continuous">
+	<!-- chester changed it to fixed -->
+        <joint name="${prefix}robotiq_85_right_inner_knuckle_joint" type="fixed">
             <parent link="${prefix}robotiq_85_base_link"/>
             <child link="${prefix}robotiq_85_right_inner_knuckle_link"/>
@@ -183,5 +189,6 @@
             </inertial>
         </link>
-        <joint name="${prefix}robotiq_85_left_finger_tip_joint" type="continuous">
+	<!-- chester changed it to fixed -->
+        <joint name="${prefix}robotiq_85_left_finger_tip_joint" type="fixed">
             <parent link="${prefix}robotiq_85_left_inner_knuckle_link"/>
             <child link="${prefix}robotiq_85_left_finger_tip_link"/>
@@ -191,5 +198,6 @@
             <mimic joint="${prefix}robotiq_85_left_knuckle_joint" multiplier="-1"/>
         </joint>
-        <joint name="${prefix}robotiq_85_right_finger_tip_joint" type="continuous">
+	<!-- chester changed it to fixed -->
+        <joint name="${prefix}robotiq_85_right_finger_tip_joint" type="fixed">
             <parent link="${prefix}robotiq_85_right_inner_knuckle_link"/>
             <child link="${prefix}robotiq_85_right_finger_tip_link"/>
